File: PCB/PiicoDev-Atmospheric-Sensor-BME280.kicad_pcb (KiCad board)
At the start: 2 copper layers, 25.4 x 25.4 mm, 29 parts, among them J1 piico, J2 piico, J3 , U1 BME280

Commit message: v11 Update
Change resistor values
Add DIP switch and remove ADR jumper
Update graphic labels
Remove solder mask between jumper pads
Update text formatting
Parts:
- removed G2: LOGO_piico, CoreElectronics_Artwork:piicodev_logo_14.2x3.4mm
- removed JP4: ADDRESS, Jumper:SolderJumper-3_P1.3mm_Bridged12_RoundedPad1.0x1.5mm
- added G1: LOGO_CoreElectronics_no-text, CoreElectronics_Artwork:CoreElectronics_logo_5mm, B.Cu at (21.8, 14.2)
- added G3: LOGO_made-with-love, CoreElectronics_Artwork:piicodev_logo_14.2x3.4mm, F.Cu at (12.7, 2.29)
- added SW1: SW_DIP_x01, CoreElectronics_Components:SW_DIP_x01_Slide_CHS-01A1, F.Cu at (22.7, 21.4)
- JP1: footprint CoreElectronics_Connectors:SolderJumper-3_P1.3mm_Closed_RoundedPad1.0x1.5mm -> CoreElectronics_Components:SolderJumper-3_P1.3mm_Closed_RoundedPad1.0x1.5mm_NumberLabels
- JP2, JP3: footprint Jumper:SolderJumper-2_P1.3mm_Bridged_RoundedPad1.0x1.5mm -> CoreElectronics_Components:SolderJumper-2_P1.3mm_Bridged_RoundedPad1.0x1.5mm
- LOGO1: footprint CoreElectronics_Logos:oshw -> CoreElectronics_Artwork:oshw
- R1, R2, R4, R5: value 4k7 -> 10k
- R3: value 1k -> 10k
- moved FID1 21.7 mm to (23.2, 7.11)
- moved FID2 21.2 mm to (1.98, 23.4)
- moved D1 5.18 mm to (2.01, 7.21), turned to 0 degrees
- moved JP3 0.67 mm to (8.29, 7.39)
- moved R3 0.30 mm to (4.34, 7.67), turned to 90 degrees
Connections:
- R5 pad 2: Net-(JP4-Pad1) -> /SDO_ADR
Routing:
- net Net-(JP4-Pad1): track 9.93 -> 0.00 mm, vias 1 -> 0
- net /SDO_ADR: track 23.0 -> 29.3 mm, vias 1 -> 3
- net GND: track 2.32 -> 3.64 mm, vias 3 -> 4
- net +3V3: track 62.3 -> 61.5 mm
- net /SCK_SCL: track 38.3 -> 39.0 mm
Other:
- board text added: "0x77 0x76"
- board text added: "ADR OFF ADR ON"
- board text added: "v11"
- board text removed: "0x76"
- board text removed: "0x77"
- board text removed: "v10"
