File: PCB/PiicoDev-Atmospheric-Sensor-BME280.kicad_pcb (KiCad board)
At the start: 2 copper layers, 25.4 x 25.4 mm, 30 parts, among them J1 piico, J2 piico, J3 , SW1 SW_DIP_x01, U1 BME280

Commit message: Rename address switch to ASW
Other:
- board text added: "ASW"
- board text added: "ASW OFF ASW ON"
- board text added: "v12"
- board text removed: "ADR"
- board text removed: "ADR OFF ADR ON"
- board text removed: "v11"
